File: eighth_brick_equivilant/DC-DC-Brick-eighth.brd (EAGLE design)
At the start: 28.6 x 87.6 mm, 20 parts

Commit message: Addressing comments and adding silk screen
Parts:
- added J1: (no value), SparkFun-Connectors:1X01
- added R5, R8: 10k, SparkFun-Resistors:0603-RES
- moved R1 0.25 mm to (7.62, 62.2)
Connections:
- new net N$8: J1.1, R5.1
- net ON/OFF: now also R5.2, R8.1
- net V-: now also R8.2
Routing:
- net N$8: track 0.00 -> 3.07 mm
- net ON/OFF: track 25.4 -> 27.8 mm
- net V+: track 22.2 -> 24.4 mm
- net GND: track 70.5 -> 72.7 mm, vias 8 -> 18
Other:
- board text added: "+12V"
- board text added: "GND"
- board text added: "ON/OFF"
- board text added: "SCL"
- board text added: "SDA"
- board text added: "Vin+"
- board text added: "Vin-"
