File: eighth_brick_equivilant/DC-DC-Brick-eighth.sch (EAGLE design)
At the start: 20 parts

Commit message: Addressing comments and adding silk screen
Parts:
- added J1: (no value), SparkFun-Connectors:CONN_01
- added R5, R8: 10k, SparkFun-Resistors:1KOHM-1/10W-1%(0603)
Connections:
- new net N$8: J1.1, R5.1
- net ON/OFF: now also R5.2, R8.1
- net V-: now also R8.2
Other:
- note added: "Pull up and pull down resistors to be used if the on/off circuitry does not work"
Changed lines of the file:
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@@
 <layer number="2" name="Route2" color="1" fill="3" visible="no" active="no"/>
 <layer number="3" name="Route3" color="4" fill="3" visible="no" active="no"/>
+<layer number="4" name="Route4" color="1" fill="4" visible="no" active="no"/>
+<layer number="5" name="Route5" color="4" fill="4" visible="no" active="no"/>
+<layer number="6" name="Route6" color="1" fill="8" visible="no" active="no"/>
+<layer number="7" name="Route7" color="4" fill="8" visible="no" active="no"/>
+<layer number="8" name="Route8" color="1" fill="2" visible="no" active="no"/>
+<layer number="9" name="Route9" color="4" fill="2" visible="no" active="no"/>
+<layer number="10" name="Route10" color="1" fill="7" visible="no" active="no"/>
+<layer number="11" name="Route11" color="4" fill="7" visible="no" active="no"/>
+<layer number="12" name="Route12" color="1" fill="5" visible="no" active="no"/>
+<layer number="13" name="Route13" color="4" fill="5" visible="no" active="no"/>
 <layer number="14" name="Route14" color="1" fill="6" visible="no" active="no"/>
 <layer number="15" name="Route15" color="4" fill="6" visible="no" active="no"/>
@@
 <layer number="230" name="230bmp" color="7" fill="1" visible="yes" active="yes"/>
 <layer number="231" name="231bmp" color="7" fill="1" visible="yes" active="yes"/>
+<layer number="232" name="Eagle3D_PG2" color="7" fill="1" visible="yes" active="yes"/>
+<layer number="233" name="Eagle3D_PG3" color="7" fill="1" visible="yes" active="yes"/>
 <layer number="248" name="Housing" color="7" fill="1" visible="yes" active="yes"/>
 <layer number="249" name="Edge" color="7" fill="1" visible="yes" active="yes"/>
@@
 <part name="P+2" library="supply1" library_urn="urn:adsk.eagle:library:371" deviceset="VCC" device=""/>
 <part name="+12V1" library="supply1" library_urn="urn:adsk.eagle:library:371" deviceset="V+" device=""/>
+<part name="R5" library="SparkFun-Resistors" deviceset="1KOHM-1/10W-1%(0603)" device="" value="10k"/>
+<part name="R8" library="SparkFun-Resistors" deviceset="1KOHM-1/10W-1%(0603)" device="" value="10k"/>
+<part name="P-3" library="supply1" library_urn="urn:adsk.eagle:library:371" deviceset="V-" device=""/>
+<part name="J1" library="SparkFun-Connectors" library_urn="urn:adsk.eagle:library:513" deviceset="CONN_01" device="" package3d_urn="urn:adsk.eagle:package:38028/1"/>
 </parts>
 <sheets>
 <sheet>
 <plain>
-<text x="205.74" y="81.28" size="1.778" layer="91">Removed pulldown res
+<text x="213.36" y="81.28" size="1.778" layer="91">Removed pulldown res
 That would cause it to
 stay on when disconnect</text>
-<text x="208.28" y="73.66" size="1.778" layer="91">Resistors (R1 and R2) values can change for each brick.</text>
+<text x="274.32" y="109.22" size="1.778" layer="91">Resistors (R1 and R2) values can change for each brick.</text>
+<text x="177.8" y="86.36" size="1.778" layer="91">Pull up and pull down
+resistors to be used
+if the on/off circuitry
+does not work</text>
 </plain>
 <instances>
@@
 <instance part="P+2" gate="VCC" x="160.02" y="66.04"/>
 <instance part="+12V1" gate="1" x="116.84" y="66.04"/>
+<instance part="R5" gate="G$1" x="205.74" y="101.6" rot="R270"/>
+<instance part="R8" gate="G$1" x="205.74" y="86.36" rot="R270"/>
+<instance part="P-3" gate="1" x="205.74" y="73.66"/>
+<instance part="J1" gate="G$1" x="195.58" y="111.76"/>
 </instances>
 <busses>
@@
 <pinref part="U$1" gate="G$1" pin="ON/!OFF1"/>
 <wire x1="231.14" y1="134.62" x2="213.36" y2="134.62" width="0.1524" layer="91"/>
-<wire x1="213.36" y1="134.62" x2="213.36" y2="91.44" width="0.1524" layer="91"/>
+<wire x1="213.36" y1="134.62" x2="213.36" y2="93.98" width="0.1524" layer="91"/>
 <label x="220.98" y="137.16" size="1.778" layer="95" rot="R180"/>
+<pinref part="R8" gate="G$1" pin="1"/>
+<pinref part="R5" gate="G$1" pin="2"/>
+<wire x1="205.74" y1="91.44" x2="205.74" y2="93.98" width="0.1524" layer="91"/>
+<wire x1="205.74" y1="93.98" x2="205.74" y2="96.52" width="0.1524" layer="91"/>
+<wire x1="205.74" y1="93.98" x2="213.36" y2="93.98" width="0.1524" layer="91"/>
+<junction x="205.74" y="93.98"/>
 </segment>
 <segment>
@@
 <wire x1="231.14" y1="154.94" x2="226.06" y2="154.94" width="0.1524" layer="91"/>
 </segment>
-</net>
+<segment>
+<pinref part="R8" gate="G$1" pin="2"/>
+<pinref part="P-3" gate="1" pin="V-"/>
+<wire x1="205.74" y1="81.28" x2="205.74" y2="76.2" width="0.1524" layer="91"/>
+</segment>
+</net>
+<net name="N$8" class="0">
+<segment>
+<pinref part="R5" gate="G$1" pin="1"/>
+<wire x1="205.74" y1="106.68" x2="205.74" y2="111.76" width="0.1524" layer="91"/>
+<pinref part="J1" gate="G$1" pin="1"/>
+<wire x1="205.74" y1="111.76" x2="203.2" y2="111.76" width="0.1524" layer="91"/>
+</segment>
+</net>
